File: Barra de luz.kicad_pcb (KiCad board)
At the start: 2 copper layers, 56.3 x 41.6 mm, 38 parts, among them J2 AVR-ISP-6, J3 Screw_Terminal_01x08, J4 VIN, SW1 SW_Push, U1 ATtiny85-20S

Commit message: adaptaciones 12V
Connections:
- J3 pad 7: GND -> +12V
Routing:
- net +12V: track 53.9 -> 104.2 mm
Changed lines of the file:
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@@
       (net 9 "/PB4") (pinfunction "Pin_6") (pintype "passive"))
     (pad "7" thru_hole circle (at 30.48 0) (size 2.6 2.6) (drill 1.3) (layers "*.Cu" "*.Mask")
-      (net 3 "GND") (pinfunction "Pin_7") (pintype "passive"))
+      (net 1 "+12V") (pinfunction "Pin_7") (pintype "passive"))
     (pad "8" thru_hole circle (at 35.56 0) (size 2.6 2.6) (drill 1.3) (layers "*.Cu" "*.Mask")
       (net 3 "GND") (pinfunction "Pin_8") (pintype "passive"))
@@
   (segment (start 122.174 99.268) (end 122.174 87.838) (width 0.762) (layer "F.Cu") (net 1))
   (segment (start 147.828 102.512) (end 143.96 106.38) (width 0.762) (layer "F.Cu") (net 1))
+  (segment (start 129.286 115.57) (end 127 113.284) (width 0.762) (layer "B.Cu") (net 1))
+  (segment (start 161.036 114.808) (end 160.274 115.57) (width 0.762) (layer "B.Cu") (net 1))
+  (segment (start 160.274 115.57) (end 129.286 115.57) (width 0.762) (layer "B.Cu") (net 1))
+  (segment (start 127 113.284) (end 127 101.046) (width 0.762) (layer "B.Cu") (net 1))
+  (segment (start 161.036 112.014) (end 161.036 114.808) (width 0.762) (layer "B.Cu") (net 1))
   (segment (start 135.416 90.346) (end 139.194 86.568) (width 0.762) (layer "F.Cu") (net 2))
   (segment (start 147.828 100.812) (end 147.828 100.792) (width 0.762) (layer "F.Cu") (net 2))
