File: Mini-85-V1.0.kicad_sch (KiCad schematic)
At the start: 8 parts, among them J2 AVR-ISP-6, J3 Screw_Terminal_01x08, SW1 SW_Push, U1 ATtiny85-20S

Commit message: feat se vrea repo
Parts:
- renumbered J3 to J1
Connections:
- net PB4: no longer J1.6 (Pin_6)
- new net +12V: J1.6 (Pin_6)
Other:
- added sheet Rele (Rele.kicad_sch)
Changed lines of the file:
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@@
+    (stroke (width 0) (type default))
+  )
+  (bus (pts (xy 12.1158 134.5692) (xy 92.8624 134.5692))
     (stroke (width 0) (type default))
   )
@@
     (stroke (width 0) (type default))
   )
+  (bus (pts (xy 92.8624 77.597) (xy 92.8624 134.5692))
+    (stroke (width 0) (type default))
+  )
   (wire (pts (xy 132.6896 51.6382) (xy 132.6896 48.387))
     (stroke (width 0) (type default))
@@
     (effects (font (size 1.27 1.27)) (justify left bottom))
   )
-  (label "PB4" (at 158.115 45.72 180) (fields_autoplaced)
-    (effects (font (size 1.27 1.27)) (justify right bottom))
+  (label "PB4" (at 61.6966 103.8606 0) (fields_autoplaced)
+    (effects (font (size 1.27 1.27)) (justify left bottom))
   )
   (label "MOSI" (at 158.115 35.56 180) (fields_autoplaced)
@@
   (symbol (lib_id "power:GND") (at 113.411 58.547 0) (unit 1)
     (in_bom yes) (on_board yes) (dnp no) (fields_autoplaced)
-    (property "Reference" "#PWR079" (at 113.411 64.897 0)
+    (property "Reference" "#PWR03" (at 113.411 64.897 0)
       (effects (font (size 1.27 1.27)) hide)
     )
@@
       (project "Barra de luz"
         (path "/25a937c4-d167-4ef2-bc5e-c2d8b81e8779"
-          (reference "#PWR079") (unit 1)
+          (reference "#PWR03") (unit 1)
         )
       )
@@
   (symbol (lib_id "power:GND") (at 132.6896 61.7982 0) (unit 1)
     (in_bom yes) (on_board yes) (dnp no) (fields_autoplaced)
-    (property "Reference" "#PWR082" (at 132.6896 68.1482 0)
+    (property "Reference" "#PWR04" (at 132.6896 68.1482 0)
       (effects (font (size 1.27 1.27)) hide)
     )
@@
       (project "Barra de luz"
         (path "/25a937c4-d167-4ef2-bc5e-c2d8b81e8779"
-          (reference "#PWR082") (unit 1)
+          (reference "#PWR04") (unit 1)
         )
       )
@@
   (symbol (lib_id "power:+5V") (at 113.411 28.067 0) (unit 1)
     (in_bom yes) (on_board yes) (dnp no)
-    (property "Reference" "#PWR076" (at 113.411 31.877 0)
+    (property "Reference" "#PWR02" (at 113.411 31.877 0)
       (effects (font (size 1.27 1.27)) hide)
     )
@@
       (project "Barra de luz"
         (path "/25a937c4-d167-4ef2-bc5e-c2d8b81e8779"
-          (reference "#PWR076") (unit 1)
+          (reference "#PWR02") (unit 1)
         )
       )
@@
   (symbol (lib_id "power:+5V") (at 221.5642 30.607 0) (unit 1)
     (in_bom yes) (on_board yes) (dnp no) (fields_autoplaced)
-    (property "Reference" "#PWR09" (at 221.5642 34.417 0)
+    (property "Reference" "#PWR08" (at 221.5642 34.417 0)
       (effects (font (size 1.27 1.27)) hide)
     )
@@
       (project "Barra de luz"
         (path "/25a937c4-d167-4ef2-bc5e-c2d8b81e8779"
-          (reference "#PWR09") (unit 1)
+          (reference "#PWR08") (unit 1)
         )
       )
@@
         (path "/25a937c4-d167-4ef2-bc5e-c2d8b81e8779"
           (reference "H1") (unit 1)
+        )
+      )
+    )
+  )
+  (symbol (lib_id "power:+12V") (at 158.115 45.72 90) (unit 1)
+    (in_bom yes) (on_board yes) (dnp no) (fields_autoplaced)
+    (property "Reference" "#PWR06" (at 161.925 45.72 0)
+      (effects (font (size 1.27 1.27)) hide)
+    )
+    (property "Value" "+12V" (at 153.6897 45.72 90)
+      (effects (font (size 1.27 1.27)) (justify left))
+    )
+    (property "Footprint" "" (at 158.115 45.72 0)
+      (effects (font (size 1.27 1.27)) hide)
+    )
+    (property "Datasheet" "" (at 158.115 45.72 0)
+      (effects (font (size 1.27 1.27)) hide)
+    )
+    (pin "1")
+    (instances
+      (project "Barra de luz"
+        (path "/25a937c4-d167-4ef2-bc5e-c2d8b81e8779"
+          (reference "#PWR06") (unit 1)
         )
       )
@@
   (symbol (lib_id "Connector:Screw_Terminal_01x08") (at 163.195 40.64 0) (unit 1)
     (in_bom yes) (on_board yes) (dnp no) (fields_autoplaced)
-    (property "Reference" "J3" (at 165.6588 40.64 0)
+    (property "Reference" "J1" (at 165.6588 40.64 0)
       (effects (font (size 1.27 1.27)) (justify left))
     )
@@
       (project "Barra de luz"
         (path "/25a937c4-d167-4ef2-bc5e-c2d8b81e8779"
-          (reference "J3") (unit 1)
+          (reference "J1") (unit 1)
         )
       )
@@
   (symbol (lib_id "power:+5V") (at 63.2206 32.8676 0) (unit 1)
     (in_bom yes) (on_board yes) (dnp no) (fields_autoplaced)
-    (property "Reference" "#PWR075" (at 63.2206 36.6776 0)
+    (property "Reference" "#PWR01" (at 63.2206 36.6776 0)
       (effects (font (size 1.27 1.27)) hide)
     )
@@
       (project "Barra de luz"
         (path "/25a937c4-d167-4ef2-bc5e-c2d8b81e8779"
-          (reference "#PWR075") (unit 1)
+          (reference "#PWR01") (unit 1)
         )
       )
@@
   (symbol (lib_id "power:GND") (at 221.5642 53.467 0) (unit 1)
     (in_bom yes) (on_board yes) (dnp no) (fields_autoplaced)
-    (property "Reference" "#PWR010" (at 221.5642 59.817 0)
+    (property "Reference" "#PWR09" (at 221.5642 59.817 0)
       (effects (font (size 1.27 1.27)) hide)
     )
@@
       (project "Barra de luz"
         (path "/25a937c4-d167-4ef2-bc5e-c2d8b81e8779"
-          (reference "#PWR010") (unit 1)
+          (reference "#PWR09") (unit 1)
         )
       )
@@
   (symbol (lib_id "power:GND") (at 158.115 50.8 0) (unit 1)
     (in_bom yes) (on_board yes) (dnp no) (fields_autoplaced)
-    (property "Reference" "#PWR012" (at 158.115 57.15 0)
+    (property "Reference" "#PWR07" (at 158.115 57.15 0)
       (effects (font (size 1.27 1.27)) hide)
     )
@@
       (project "Barra de luz"
         (path "/25a937c4-d167-4ef2-bc5e-c2d8b81e8779"
-          (reference "#PWR012") (unit 1)
+          (reference "#PWR07") (unit 1)
         )
       )
@@
   (symbol (lib_id "power:+5V") (at 158.115 33.02 0) (unit 1)
     (in_bom yes) (on_board yes) (dnp no)
-    (property "Reference" "#PWR011" (at 158.115 36.83 0)
+    (property "Reference" "#PWR05" (at 158.115 36.83 0)
       (effects (font (size 1.27 1.27)) hide)
     )
@@
       (project "Barra de luz"
         (path "/25a937c4-d167-4ef2-bc5e-c2d8b81e8779"
-          (reference "#PWR011") (unit 1)
-        )
-      )
-    )
+          (reference "#PWR05") (unit 1)
+        )
+      )
+    )
+  )
+  (sheet (at 41.9862 98.933) (size 19.7104 13.6652) (fields_autoplaced)
+    (stroke (width 0.1524) (type solid))
+    (fill (color 0 0 0 0.0000))
+    (property "Sheetname" "Rele" (at 41.9862 98.2214 0)
+      (effects (font (size 1.27 1.27)) (justify left bottom))
+    )
+    (property "Sheetfile" "Rele.kicad_sch" (at 41.9862 113.1828 0)
+      (effects (font (size 1.27 1.27)) (justify left top))
+    )
+    (pin "sig" input (at 61.6966 103.8606 0)
+      (effects (font (size 1.27 1.27)) (justify right))
+    )
+    (instances
+      (project "Barra de luz"
+        (path "/25a937c4-d167-4ef2-bc5e-c2d8b81e8779" (page "3"))
+      )
+    )
