File: Regulador.kicad_sch (KiCad schematic)
At the start: 11 parts, among them J1 Conn_01x02_Pin

Commit message: ajustes para quitar leds y hacer placa mas sencilla
Parts:
- removed J1: Conn_01x02_Pin, Connector_PinHeader_2.54mm:PinHeader_1x02_P2.54mm_Vertical, symbol Connector:Conn_01x02_Pin
- added J4: VIN, TerminalBlock_Phoenix:TerminalBlock_Phoenix_MKDS-3-2-5.08_1x02_P5.08mm_Horizontal, symbol Connector:Screw_Terminal_01x02
Connections:
- net +12V: now also J4.2 (Pin_2)
- net GND: now also J4.1 (Pin_1)
Changed lines of the file:
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@@
-    )
-  )
-  (symbol (lib_id "Connector:Conn_01x02_Pin") (at 99.9744 91.4908 0) (unit 1)
-    (in_bom yes) (on_board yes) (dnp no) (fields_autoplaced)
-    (property "Reference" "J1" (at 100.6094 86.371 0)
-      (effects (font (size 1.27 1.27)))
-    )
-    (property "Value" "Conn_01x02_Pin" (at 100.6094 88.911 0)
-      (effects (font (size 1.27 1.27)))
-    )
-    (property "Footprint" "Connector_PinHeader_2.54mm:PinHeader_1x02_P2.54mm_Vertical" (at 99.9744 91.4908 0)
-      (effects (font (size 1.27 1.27)) hide)
-    )
-    (property "Datasheet" "~" (at 99.9744 91.4908 0)
-      (effects (font (size 1.27 1.27)) hide)
-    )
-    (pin "1")
-    (pin "2")
-    (instances
-      (project "Barra de luz"
-        (path "/25a937c4-d167-4ef2-bc5e-c2d8b81e8779/9766723e-22df-4d3c-ad55-2258ea78ff30"
-          (reference "J1") (unit 1)
-        )
-      )
     )
   )
@@
         )
       )
+    )
+  )
+  (symbol (lib_id "Connector:Screw_Terminal_01x02") (at 99.9744 94.0308 180) (unit 1)
+    (in_bom yes) (on_board yes) (dnp no)
+    (property "Reference" "J4" (at 97.2897 94.0308 0)
+      (effects (font (size 1.27 1.27)) (justify left))
+    )
+    (property "Value" "VIN" (at 113.2409 85.4664 0)
+      (effects (font (size 1.27 1.27)) (justify left) hide)
+    )
+    (property "Footprint" "TerminalBlock_Phoenix:TerminalBlock_Phoenix_MKDS-3-2-5.08_1x02_P5.08mm_Horizontal" (at 99.9744 94.0308 0)
+      (effects (font (size 1.27 1.27)) hide)
+    )
+    (property "Datasheet" "~" (at 99.9744 94.0308 0)
+      (effects (font (size 1.27 1.27)) hide)
+    )
+    (pin "1")
+    (pin "2")
+    (instances
+      (project "Barra de luz"
+        (path "/25a937c4-d167-4ef2-bc5e-c2d8b81e8779/9766723e-22df-4d3c-ad55-2258ea78ff30"
+          (reference "J4") (unit 1)
+        )
+      )

Commit message: feat se vrea repo
Parts:
- renumbered J4 to J3
Changed lines of the file:
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@@
   (symbol (lib_id "power:GND") (at 168.3004 108.0008 0) (unit 1)
     (in_bom yes) (on_board yes) (dnp no) (fields_autoplaced)
-    (property "Reference" "#PWR06" (at 168.3004 114.3508 0)
+    (property "Reference" "#PWR015" (at 168.3004 114.3508 0)
       (effects (font (size 1.27 1.27)) hide)
     )
@@
       (project "Barra de luz"
         (path "/25a937c4-d167-4ef2-bc5e-c2d8b81e8779/9766723e-22df-4d3c-ad55-2258ea78ff30"
-          (reference "#PWR06") (unit 1)
+          (reference "#PWR015") (unit 1)
         )
       )
@@
   (symbol (lib_id "power:GND") (at 187.3504 108.0008 0) (unit 1)
     (in_bom yes) (on_board yes) (dnp no) (fields_autoplaced)
-    (property "Reference" "#PWR08" (at 187.3504 114.3508 0)
+    (property "Reference" "#PWR017" (at 187.3504 114.3508 0)
       (effects (font (size 1.27 1.27)) hide)
     )
@@
       (project "Barra de luz"
         (path "/25a937c4-d167-4ef2-bc5e-c2d8b81e8779/9766723e-22df-4d3c-ad55-2258ea78ff30"
-          (reference "#PWR08") (unit 1)
+          (reference "#PWR017") (unit 1)
         )
       )
@@
   (symbol (lib_id "power:+12V") (at 115.2144 83.1088 0) (unit 1)
     (in_bom yes) (on_board yes) (dnp no) (fields_autoplaced)
-    (property "Reference" "#PWR02" (at 115.2144 86.9188 0)
+    (property "Reference" "#PWR011" (at 115.2144 86.9188 0)
       (effects (font (size 1.27 1.27)) hide)
     )
@@
       (project "Barra de luz"
         (path "/25a937c4-d167-4ef2-bc5e-c2d8b81e8779/9766723e-22df-4d3c-ad55-2258ea78ff30"
-          (reference "#PWR02") (unit 1)
+          (reference "#PWR011") (unit 1)
         )
       )
@@
   (symbol (lib_id "power:GND") (at 105.0798 102.7176 0) (unit 1)
     (in_bom yes) (on_board yes) (dnp no) (fields_autoplaced)
-    (property "Reference" "#PWR01" (at 105.0798 109.0676 0)
+    (property "Reference" "#PWR010" (at 105.0798 109.0676 0)
       (effects (font (size 1.27 1.27)) hide)
     )
@@
       (project "Barra de luz"
         (path "/25a937c4-d167-4ef2-bc5e-c2d8b81e8779/9766723e-22df-4d3c-ad55-2258ea78ff30"
-          (reference "#PWR01") (unit 1)
+          (reference "#PWR010") (unit 1)
         )
       )
@@
   (symbol (lib_id "power:GND") (at 182.3974 89.9414 0) (unit 1)
     (in_bom yes) (on_board yes) (dnp no) (fields_autoplaced)
-    (property "Reference" "#PWR07" (at 182.3974 96.2914 0)
+    (property "Reference" "#PWR016" (at 182.3974 96.2914 0)
       (effects (font (size 1.27 1.27)) hide)
     )
@@
       (project "Barra de luz"
         (path "/25a937c4-d167-4ef2-bc5e-c2d8b81e8779/9766723e-22df-4d3c-ad55-2258ea78ff30"
-          (reference "#PWR07") (unit 1)
+          (reference "#PWR016") (unit 1)
         )
       )
@@
   (symbol (lib_id "power:GND") (at 151.7904 106.7308 0) (unit 1)
     (in_bom yes) (on_board yes) (dnp no) (fields_autoplaced)
-    (property "Reference" "#PWR05" (at 151.7904 113.0808 0)
+    (property "Reference" "#PWR014" (at 151.7904 113.0808 0)
       (effects (font (size 1.27 1.27)) hide)
     )
@@
       (project "Barra de luz"
         (path "/25a937c4-d167-4ef2-bc5e-c2d8b81e8779/9766723e-22df-4d3c-ad55-2258ea78ff30"
-          (reference "#PWR05") (unit 1)
+          (reference "#PWR014") (unit 1)
         )
       )
@@
   (symbol (lib_id "power:GND") (at 115.2144 108.0008 0) (unit 1)
     (in_bom yes) (on_board yes) (dnp no) (fields_autoplaced)
-    (property "Reference" "#PWR03" (at 115.2144 114.3508 0)
+    (property "Reference" "#PWR012" (at 115.2144 114.3508 0)
       (effects (font (size 1.27 1.27)) hide)
     )
@@
       (project "Barra de luz"
         (path "/25a937c4-d167-4ef2-bc5e-c2d8b81e8779/9766723e-22df-4d3c-ad55-2258ea78ff30"
-          (reference "#PWR03") (unit 1)
+          (reference "#PWR012") (unit 1)
         )
       )
@@
   (symbol (lib_id "Connector:Screw_Terminal_01x02") (at 99.9744 94.0308 180) (unit 1)
     (in_bom yes) (on_board yes) (dnp no)
-    (property "Reference" "J4" (at 97.2897 94.0308 0)
+    (property "Reference" "J3" (at 97.2897 94.0308 0)
       (effects (font (size 1.27 1.27)) (justify left))
     )
@@
       (project "Barra de luz"
         (path "/25a937c4-d167-4ef2-bc5e-c2d8b81e8779/9766723e-22df-4d3c-ad55-2258ea78ff30"
-          (reference "J4") (unit 1)
+          (reference "J3") (unit 1)
         )
       )
@@
   (symbol (lib_id "power:GND") (at 130.2004 102.9208 0) (unit 1)
     (in_bom yes) (on_board yes) (dnp no) (fields_autoplaced)
-    (property "Reference" "#PWR04" (at 130.2004 109.2708 0)
+    (property "Reference" "#PWR013" (at 130.2004 109.2708 0)
       (effects (font (size 1.27 1.27)) hide)
     )
@@
       (project "Barra de luz"
         (path "/25a937c4-d167-4ef2-bc5e-c2d8b81e8779/9766723e-22df-4d3c-ad55-2258ea78ff30"
-          (reference "#PWR04") (unit 1)
-        )
-      )
+          (reference "#PWR013") (unit 1)
+        )
+      )
